File: Section A - Title A.kicad_sch (KiCad schematic)
At the start: 0 parts

Commit message: First draft of the schematic
Parts:
- added C1, C2: 100uF, Capacitor_THT:CP_Radial_D7.5mm_P2.50mm, symbol Device:C_Polarized
- added H1, H2, H3, H4: MountingHole_Pad_MP, MountingHole:MountingHole_3.2mm_M3_DIN965_Pad, symbol Mechanical:MountingHole_Pad_MP
- added J10: Conn_01x26, Connector_Dsub:DSUB-26-HD_Socket_Horizontal_P2.29x2.54mm_EdgePinOffset8.35mm_Housed_MountingHolesOffset10.89mm, symbol Connector_Generic:Conn_01x26
- added J11: L17HTHES4R1C, L17HTHES4R1C, symbol SamacSys_Parts:L17HTHES4R1C
- added J12: DA15_Socket_MountingHoles, Connector_Dsub:DSUB-15-HD_Pins_Horizontal_P2.29x1.90mm_EdgePinOffset3.03mm_Housed_MountingHolesOffset4.94mm, symbol Connector:DA15_Socket_MountingHoles
- added J13: FCR7350R, FCR7350R, symbol SamacSys_Parts:FCR7350R
- added J14: FCR7350B, FCR7350B, symbol SamacSys_Parts:FCR7350B
- added J15: DE09-SL-24, DE09SL24, symbol SamacSys_Parts:DE09-SL-24
- added J25: KLDX-0202-A-LT, KLDX0202ALT, symbol SamacSys_Parts:KLDX-0202-A-LT
- added JP2: Jumper_3_Open, Connector_PinHeader_2.54mm:PinHeader_1x03_P2.54mm_Vertical, symbol Jumper:Jumper_3_Open
- added Q3: IRLZ44N, Package_TO_SOT_THT:TO-220-3_Horizontal_TabDown, symbol Transistor_FET:IRLZ44N
- added R33, R34, R35, R36, R38, R39, R40, R41: 100R, Resistor_SMD:R_0805_2012Metric, symbol Device:R
- added R65: 10K, Resistor_SMD:R_0805_2012Metric, symbol Device:R
- added SW1: SW_Rotary_1x9_MP, SamacSys_Parts:CK1059, symbol SamacSys_Parts:SW_Rotary_1x12
- added T7, T8, VC1, VC2, VC3, VC4, VC5, VC6: TestPoint, SamacSys_Parts:TestPoint_Pad_0.6x0.6mm, symbol Connector:TestPoint
- added VTX1, VTX2: TestPoint, TestPoint:TestPoint_Pad_1.0x1.0mm, symbol Connector:TestPoint
Connections:
- new net: J11.8, R35.2
- new net: Q3.1 (G), R41.2, R65.1
- new net: J11.10, R38.1
- new net: J11.5, R34.2
- new net: J11.12, R39.1
- new net: J11.14, R40.1
- new net: J11.4, R33.2
- new net: J11.9, R36.2
- new net: J14.1, Q3.2 (D)
- new net: J14.2, J14.3, J14.4, J14.5
- new net: J13.2, J13.3, J13.4, J13.5
- new net +5V: JP2.1 (A)
- new net DL_1_IN: J15.2
- new net DL_1_OUT: J15.7
- new net DL_2_IN: J15.3
- new net DL_2_OUT: J15.8
- new net DL_3_IN: J15.4
- new net DL_3_OUT: J15.9
- new net EL: R41.1
- new net EXT_5V: J25.1, JP2.3 (B)
- new net GND: C1.2, C2.2, J10.11 (Pin_11), J10.12 (Pin_12), J10.13 (Pin_13), J10.14 (Pin_14), J10.15 (Pin_15), J10.16 (Pin_16), J10.17 (Pin_17), J10.18 (Pin_18), J10.19 (Pin_19), J10.26 (Pin_26), J10.3 (Pin_3), J11.11, J11.2, J11.3, J11.7, J15.1, J15.5, J15.6, J25.2, J25.3, Q3.3 (S), R65.2
- new net LD9_5V: J10.25 (Pin_25), SW1.10, T8.1
- new net RX: R39.2
- new net Relay_VCC: C1.1, C2.1, JP2.2 (C)
- new net Selector Out: J13.1, SW1.A1
- new net TTL1: R33.1
- new net TTL2: R34.1
- new net TTL3: R36.1
- new net TTL4: R38.2
- new net TTL5: R40.2
- new net TX: R35.1
- new net VCAM_1 +28V: J10.4 (Pin_4), SW1.3, VC1.1
- new net VCAM_2 +28V: J10.5 (Pin_5), SW1.4, VC2.1
- new net VCAM_3 +28V: J10.6 (Pin_6), SW1.5, VC3.1
- new net VCAM_4 +28V: J10.7 (Pin_7), SW1.6, VC4.1
- new net VCAM_5 +28V: J10.8 (Pin_8), SW1.7, VC5.1
- new net VCAM_6 +28V: J10.9 (Pin_9), SW1.8, VC6.1
- new net VDCU_28V: J11.1, J11.6, SW1.9, T7.1
- new net VTX_1_28V: J10.1 (Pin_1), SW1.1, VTX1.1
- new net VTX_2_28V: J10.2 (Pin_2), SW1.2, VTX2.1
- no-connect marks 0 -> 34
Other:
- note added: "* Indicates a PWM-capable pin"
- note added: "Connects to PDCU J2 HDC9S3S00S/AA"
- note added: "Connects to PDCU J4 DD15S3S00S/AA"
- note added: "Connects to PDCU J5 DD26S3S00S/AA"
- note added: "Electronic Load"
- note added: "J3 DD15M3S00S/AA"
- note added: "Selector Switch"
