File: Section B - TItle B.kicad_sch (KiCad schematic)
At the start: 0 parts

Commit message: First draft of the schematic
Parts:
- added C34, C35, C36, C37: 100n, Capacitor_SMD:C_0603_1608Metric, symbol Device:C
- added DL1, DL2, DL3, TTL1, TTL2, TTL3, TTL4, TTL5: TestPoint, TestPoint:TestPoint_Pad_1.0x1.0mm, symbol Connector:TestPoint
- added J1: Power, Connector_PinHeader_2.54mm:PinHeader_1x08_P2.54mm_Vertical, symbol Connector_Generic:Conn_01x08
- added J16, J17, J18, J19, J20, J21, J22, J23, J24, J5: OSTOQ025450, SHDR2W100P0X508_1X2_1216X860X1230P, symbol SamacSys_Parts:OSTOQ025450
- added J2, J3: Analog, Connector_PinHeader_2.54mm:PinHeader_1x08_P2.54mm_Vertical, symbol Connector_Generic:Conn_01x08
- added J4: Digital, Connector_PinHeader_2.54mm:PinHeader_2x18_P2.54mm_Vertical, symbol Connector_Generic:Conn_02x18_Odd_Even
- added J6: PWM, Connector_PinHeader_2.54mm:PinHeader_1x10_P2.54mm_Vertical, symbol Connector_Generic:Conn_01x10
- added J7: PWM, Connector_PinHeader_2.54mm:PinHeader_1x08_P2.54mm_Vertical, symbol Connector_Generic:Conn_01x08
- added J8: Communication, Connector_PinHeader_2.54mm:PinHeader_1x08_P2.54mm_Vertical, symbol Connector_Generic:Conn_01x08
- added J9: Conn_01x06, Connector_PinHeader_2.54mm:PinHeader_1x06_P2.54mm_Vertical, symbol Connector_Generic:Conn_01x06
- added K1, K10, K2, K3, K4, K5, K6, K7, K8, K9: OJE-SH-105LMH,000, OJESH105LMH000, symbol SamacSys_Parts:OJE-SH-105LMH,000
- added K11, K12, K13, K14, K15, K16, K17, K18, K19, K20: VOR1003M4T, VOR1003M4T, symbol SamacSys_Parts:VOR1003M4T
- added Q1, Q10, Q11, Q12, Q13, Q14, Q15, Q16, Q17, Q2, Q22, Q23, Q24, Q28, Q29, Q31, Q33, Q4, Q9: IRLML2060, Package_TO_SOT_SMD:SOT-23, symbol Transistor_FET:IRLML2060
- added Q27, Q30, Q32, Q34: DMP6185SEQ-13, SOT230P700X180-4N, symbol SamacSys_Parts:DMP6185SEQ-13
- added R1, R10, R102, R103, R104, R2, R3, R4, R5, R56, R57, R6, R62, R7, R8, R9: 100R, Resistor_SMD:R_0805_2012Metric, symbol Device:R
- added R109, R110, R113, R114, R116, R117, R119, R120, R66, R67, R68, R69, R70, R71, R72, R73, R74, R75: 10K, Resistor_SMD:R_0805_2012Metric, symbol Device:R
- added R11, R13, R15, R17, R19, R21, R23, R25, R27, R29, R42, R43, R44: 100K, Resistor_SMD:R_0805_2012Metric, symbol Device:R
- added R111, R112, R115, R118: 2K, Resistor_SMD:R_0805_2012Metric, symbol Device:R
- added R12, R14, R16, R18, R20, R22, R24, R26, R28, R30: 22K, Resistor_SMD:R_0805_2012Metric, symbol Device:R
- added R31, R32, R37: R, Resistor_SMD:R_0805_2012Metric, symbol Device:R
- added R76, R77, R78, R79, R80, R81, R82, R83, R84, R85: 750R, Resistor_SMD:R_0805_2012Metric, symbol Device:R
Connections:
- new net: Q22.1 (G), R44.1, R62.2
- new net: Q29.3 (D), Q30.1 (G), R113.1, R114.1
- new net: Q31.3 (D), Q32.1 (G), R116.1, R117.1
- new net: K18.1 (A), R83.1
- new net: Q2.1 (G), R37.2
- new net: Q4.1 (G), R43.1, R56.1
- new net: Q33.3 (D), Q34.1 (G), R119.1, R120.1
- new net: Q13.1 (G), R42.1, R57.1
- new net: K16.1 (A), R81.1
- new net: K17.1 (A), R82.1
- new net: Q27.1 (G), Q28.3 (D), R109.1, R110.1
- new net: K13.1 (A), R78.1
- new net: K14.1 (A), R79.1
- new net: K15.1 (A), R80.1
- new net *10: J6.8 (Pin_8), R8.1
- new net *11: J6.7 (Pin_7), R7.1
- new net *12: J6.6 (Pin_6), R6.1
- new net *13: J6.5 (Pin_5), R5.1
- new net *2: J7.6 (Pin_6), R104.1
- new net *3: J7.5 (Pin_5), R103.1
- new net *4: J7.4 (Pin_4), R4.1
- new net *44: J4.11 (Pin_11)
- new net *46: J4.9 (Pin_9)
- new net *5: J7.3 (Pin_3), R3.1
- new net *6: J7.2 (Pin_2), R2.1
- new net *7: J7.1 (Pin_1), R1.1
- new net *8: J6.10 (Pin_10), R10.1
- new net *9: J6.9 (Pin_9), R9.1
- new net +3V3: J1.4 (Pin_4)
- new net +5V: J1.5 (Pin_5), J4.35 (Pin_35), J4.36 (Pin_36), Q1.3 (D), Q2.3 (D)
- new net 22: J4.33 (Pin_33), R102.1
- new net 24: J4.31 (Pin_31)
- new net 26: J4.29 (Pin_29)
- new net 28: J4.27 (Pin_27)
- new net 32: J4.23 (Pin_23)
- new net 42: J4.13 (Pin_13)
- new net 48: J4.7 (Pin_7)
- new net 50: J4.5 (Pin_5)
- new net A: R103.2
- new net A0: J2.1 (Pin_1), R29.1, R30.1
- new net A1: J2.2 (Pin_2), R27.1, R28.1
- new net A10: J3.3 (Pin_3)
- new net A11: J3.4 (Pin_4)
- new net A12: J3.5 (Pin_5)
- new net A13: J3.6 (Pin_6)
- new net A14: J3.7 (Pin_7)
- new net A15: J3.8 (Pin_8)
- new net A2: J2.3 (Pin_3), R25.1, R26.1
- new net A3: J2.4 (Pin_4), R23.1, R24.1
- new net A4: J2.5 (Pin_5), R21.1, R22.1
- new net A5: J2.6 (Pin_6), R19.1, R20.1
- new net A6: J2.7 (Pin_7), R17.1, R18.1
- new net A7: J2.8 (Pin_8), R15.1, R16.1
- new net A8: J3.1 (Pin_1), R13.1, R14.1
- new net A9: J3.2 (Pin_2), R11.1, R12.1
- new net AREF: J6.3 (Pin_3)
- new net Ardu_RX: J8.2 (Pin_2), Q1.2 (S), R31.2
- new net B: R104.2
- new net C: R102.2
- new net C_K1: K1.2 (COIL_2), Q12.3 (D)
- new net C_K10: K8.2 (COIL_2), Q23.3 (D)
- new net C_K2: K2.2 (COIL_2), Q11.3 (D)
- new net C_K3: K3.2 (COIL_2), Q9.3 (D)
- new net C_K4: K4.2 (COIL_2), Q10.3 (D)
- new net C_K5: K5.2 (COIL_2), Q16.3 (D)
- new net C_K6: K7.2 (COIL_2), Q17.3 (D)
- new net C_K7: K9.2 (COIL_2), Q14.3 (D)
- new net C_K8: K10.2 (COIL_2), Q15.3 (D)
- new net C_K9: K6.2 (COIL_2), Q24.3 (D)
- new net DL1: DL1.1, J4.4 (Pin_4), R56.2
- new net DL2: DL2.1, J4.6 (Pin_6), R57.2
- new net DL3: DL3.1, J4.8 (Pin_8), R62.1
- new net DL_1_IN: Q4.3 (D)
- new net DL_1_OUT: Q4.2 (S), R43.2
- new net DL_2_IN: Q13.3 (D)
- new net DL_2_OUT: Q13.2 (S), R42.2
- new net DL_3_IN: Q22.3 (D)
- new net DL_3_OUT: Q22.2 (S), R44.2
- new net EL: J4.3 (Pin_3)
- new net GND: C34.2, C35.2, C36.2, C37.2, J1.6 (Pin_6), J1.7 (Pin_7), J16.1, J17.1, J18.1, J19.1, J20.1, J21.1, J22.1, J23.1, J24.1, J4.1 (Pin_1), J4.2 (Pin_2), J5.1, J6.4 (Pin_4), K11.2 (K), K12.2 (K), K13.2 (K), K14.2 (K), K15.2 (K), K16.2 (K), K17.2 (K), K18.2 (K), K19.2 (K), K20.2 (K), Q10.2 (S), Q11.2 (S), Q12.2 (S), Q14.2 (S), Q15.2 (S), Q16.2 (S), Q17.2 (S), Q23.2 (S), Q24.2 (S), Q28.2 (S), Q29.2 (S), Q31.2 (S), Q33.2 (S), Q9.2 (S), R111.2, R112.2, R115.2, R118.2, R12.2, R14.2, R16.2, R18.2, R20.2, R22.2, R24.2, R26.2, R28.2, R30.2, R31.1, R32.1, R66.2, R67.2, R68.2, R69.2, R70.2, R71.2, R72.2, R73.2, R74.2, R75.2
- new net IOREF: J1.2 (Pin_2)
- new net K1: Q12.1 (G), R4.2, R66.1
- new net K10: Q23.1 (G), R5.2, R75.1
- new net K10_No: J17.2, K10.4 (NO)
- new net K11: J4.15 (Pin_15), R76.2
- new net K11_1: C36.1, K11.1 (A), Q31.1 (G), R115.1, R76.1
- new net K12: J4.16 (Pin_16), R77.2
- new net K12_1: C37.1, K12.1 (A), Q33.1 (G), R118.1, R77.1
- new net K13: J4.17 (Pin_17), R78.2
- new net K14: J4.18 (Pin_18), R79.2
- new net K15: J4.19 (Pin_19), R80.2
- new net K16: J4.20 (Pin_20), R81.2
- new net K17: J4.21 (Pin_21), R82.2
- new net K18: J4.22 (Pin_22), R83.2
- new net K19: J4.25 (Pin_25), R84.2
- new net K19_1: C34.1, K19.1 (A), Q28.1 (G), R111.1, R84.1
- new net K1_No: J24.2, K1.4 (NO)
- new net K2: Q11.1 (G), R3.2, R67.1
- new net K20: J4.24 (Pin_24), R85.2
- new net K20_1: C35.1, K20.1 (A), Q29.1 (G), R112.1, R85.1
- new net K2_No: J23.2, K2.4 (NO)
- new net K3: Q9.1 (G), R2.2, R68.1
- new net K3_No: J22.2, K3.4 (NO)
- new net K4: Q10.1 (G), R1.2, R69.1
- new net K4_No: J21.2, K4.4 (NO)
- new net K5: Q16.1 (G), R10.2, R70.1
- new net K5_No: J20.2, K5.4 (NO)
- new net K6: Q17.1 (G), R71.1, R9.2
- new net K6_No: J16.2, K6.4 (NO)
- new net K7: Q14.1 (G), R72.1, R8.2
- new net K7_No: J19.2, K7.4 (NO)
- new net K8: Q15.1 (G), R7.2, R73.1
- new net K8_No: J5.2, K8.4 (NO)
- new net K9: Q24.1 (G), R6.2, R74.1
- new net K9_No: J18.2, K9.4 (NO)
- new net LD9_5V: K20.3 (S2), K8.3 (COM), Q30.3 (S), R11.2, R113.2, R114.2
- new net RESET: J1.3 (Pin_3)
- new net RX: Q2.2 (S), R32.2
- new net RX0/0: J7.8 (Pin_8)
- new net RX1/19: J8.6 (Pin_6), J9.4 (Pin_4)
- new net RX2/17: J8.4 (Pin_4), J9.2 (Pin_2)
- new net Relay_VCC: K1.1 (COIL_1), K10.1 (COIL_1), K2.1 (COIL_1), K3.1 (COIL_1), K4.1 (COIL_1), K5.1 (COIL_1), K6.1 (COIL_1), K7.1 (COIL_1), K8.1 (COIL_1), K9.1 (COIL_1)
- new net SCL/21: J6.1 (Pin_1), J8.8 (Pin_8), J9.6 (Pin_6)
- new net SDA/20: J6.2 (Pin_2), J8.7 (Pin_7), J9.5 (Pin_5)
- new net Selector Out: K11.4 (S1), K12.4 (S1), K13.4 (S1), K14.4 (S1), K15.4 (S1), K16.4 (S1), K17.4 (S1), K18.4 (S1), K19.4 (S1), K20.4 (S1), Q27.4 (D_2), Q30.4 (D_2), Q32.4 (D_2), Q34.4 (D_2)
- new net TTL1: J4.30 (Pin_30), TTL1.1
- new net TTL2: J4.32 (Pin_32), TTL2.1
- new net TTL3: J4.28 (Pin_28), TTL3.1
- new net TTL4: J4.34 (Pin_34), TTL4.1
- new net TTL5: J4.26 (Pin_26), TTL5.1
- new net TX: Q1.1 (G)
- new net TX0/1: J7.7 (Pin_7)
- new net TX1/18: J8.5 (Pin_5), J9.3 (Pin_3)
- new net TX2/16: J8.3 (Pin_3), J9.1 (Pin_1)
- new net TX3/14: J8.1 (Pin_1), R37.1
- new net VCAM_1 +28V: K13.3 (S2), K3.3 (COM), R25.2
- new net VCAM_2 +28V: K14.3 (S2), K4.3 (COM), R23.2
- new net VCAM_3 +28V: K15.3 (S2), K5.3 (COM), R21.2
- new net VCAM_4 +28V: K16.3 (S2), K7.3 (COM), R19.2
- new net VCAM_5 +28V: K17.3 (S2), K9.3 (COM), R17.2
- new net VCAM_6 +28V: K10.3 (COM), K18.3 (S2), R15.2
- new net VCC: J1.8 (Pin_8)
- new net VDCU_28V: K19.3 (S2), K6.3 (COM), Q27.3 (S), R109.2, R110.2, R13.2
- new net VTX_1_28V: K1.3 (COM), K11.3 (S2), Q32.3 (S), R116.2, R117.2, R29.2
- new net VTX_2_28V: K12.3 (S2), K2.3 (COM), Q34.3 (S), R119.2, R120.2, R27.2
- no-connect marks 0 -> 28
Other:
- note added: "*44"
- note added: "*45"
- note added: "*46"
- note added: "*52"
- note added: "22"
- note added: "23"
- note added: "24"
- note added: "25"
- note added: "26"
- note added: "27"
- note added: "28"
- note added: "29"
- note added: "30"
- note added: "31"
- note added: "32"
- note added: "33"
- note added: "34"
- note added: "35"
- note added: "36"
- note added: "37"
- note added: "38"
- note added: "39"
- note added: "40"
- note added: "41"
- note added: "42"
- note added: "43"
- note added: "47"
- note added: "48"
- note added: "49"
- note added: "50"
- note added: "51"
- note added: "53"
- note added: "A0"
- note added: "A1"
- note added: "A2"
- note added: "A3"
- note added: "A4"
- note added: "A5"
- note added: "A6"
- note added: "A7"
- note added: "A8"
- note added: "A9"
- note added: "From VDCU"
- note added: "Vin"
