File: REALTRA_TRIAL.kicad_pcb (KiCad board)
At the start: 6 copper layers, 0 parts

Commit message: First draft of PCB Preliminary version
Parts:
- added C1: 100uF, Capacitor_THT:CP_Radial_D7.5mm_P2.50mm, F.Cu at (336.0, 187.3)
- added C2: 100uF, Capacitor_THT:CP_Radial_D7.5mm_P2.50mm, F.Cu at (345.8, 187.3)
- added C34: 100n, Capacitor_SMD:C_0603_1608Metric, B.Cu at (167.0, 146.0)
- added C35: 100n, Capacitor_SMD:C_0603_1608Metric, B.Cu at (175.5, 146.0)
- added C36: 100n, Capacitor_SMD:C_0603_1608Metric, B.Cu at (228.5, 143.2)
- added C37: 100n, Capacitor_SMD:C_0603_1608Metric, B.Cu at (220.5, 143.2)
- added DL1: TestPoint, TestPoint:TestPoint_Pad_1.0x1.0mm, F.Cu at (185.9, 173.0)
- added DL2: TestPoint, TestPoint:TestPoint_Pad_1.0x1.0mm, F.Cu at (179.2, 173.0)
- added DL3: TestPoint, TestPoint:TestPoint_Pad_1.0x1.0mm, F.Cu at (172.2, 173.0)
- added H1: MountingHole_Pad_MP, MountingHole:MountingHole_3.2mm_M3_DIN965_Pad, F.Cu at (54.0, 196.0)
- added H2: MountingHole_Pad_MP, MountingHole:MountingHole_3.2mm_M3_DIN965_Pad, F.Cu at (366.0, 196.0)
- added H3: MountingHole_Pad_MP, MountingHole:MountingHole_3.2mm_M3_DIN965_Pad, F.Cu at (54.0, 54.0)
- added H4: MountingHole_Pad_MP, MountingHole:MountingHole_3.2mm_M3_DIN965_Pad, F.Cu at (366.0, 54.0)
- added J1: Power, Connector_PinHeader_2.54mm:PinHeader_1x08_P2.54mm_Vertical, F.Cu at (323.7, 161.9)
- added J10: Conn_01x26, Connector_Dsub:DSUB-26-HD_Socket_Horizontal_P2.29x2.54mm_EdgePinOffset8.35mm_Housed_MountingHolesOffset10.89mm, F.Cu at (239.4, 186.5)
- added J11: L17HTHES4R1C, SamacSys_Parts:L17HTHES4R1C, F.Cu at (134.0, 186.0)
- added J12: DA15_Socket_MountingHoles, Connector_Dsub:DSUB-15-HD_Pins_Horizontal_P2.29x1.90mm_EdgePinOffset3.03mm_Housed_MountingHolesOffset4.94mm, F.Cu at (361.0, 92.2)
- added J13: FCR7350R, SamacSys_Parts:FCR7350R, F.Cu at (94.4, 186.5)
- added J14: FCR7350B, SamacSys_Parts:FCR7350B, F.Cu at (74.4, 186.5)
- added J15: DE09-SL-24, SamacSys_Parts:DE09SL24, F.Cu at (185.9, 188.5)
- added J16: OSTOQ025450, SamacSys_Parts:SHDR2W100P0X508_1X2_1216X860X1230P, F.Cu at (271.0, 55.0)
- added J17: OSTOQ025450, SamacSys_Parts:SHDR2W100P0X508_1X2_1216X860X1230P, F.Cu at (246.0, 55.0)
- added J18: OSTOQ025450, SamacSys_Parts:SHDR2W100P0X508_1X2_1216X860X1230P, F.Cu at (221.0, 55.0)
- added J19: OSTOQ025450, SamacSys_Parts:SHDR2W100P0X508_1X2_1216X860X1230P, F.Cu at (196.0, 55.0)
- added J2: Analog, Connector_PinHeader_2.54mm:PinHeader_1x08_P2.54mm_Vertical, F.Cu at (300.8, 161.9)
- added J20: OSTOQ025450, SamacSys_Parts:SHDR2W100P0X508_1X2_1216X860X1230P, F.Cu at (171.0, 55.0)
- added J21: OSTOQ025450, SamacSys_Parts:SHDR2W100P0X508_1X2_1216X860X1230P, F.Cu at (146.0, 55.0)
- added J22: OSTOQ025450, SamacSys_Parts:SHDR2W100P0X508_1X2_1216X860X1230P, F.Cu at (121.0, 55.0)
- added J23: OSTOQ025450, SamacSys_Parts:SHDR2W100P0X508_1X2_1216X860X1230P, F.Cu at (96.0, 55.0)
- added J24: OSTOQ025450, SamacSys_Parts:SHDR2W100P0X508_1X2_1216X860X1230P, F.Cu at (71.0, 55.0)
- added J25: KLDX-0202-A-LT, SamacSys_Parts:KLDX0202ALT, F.Cu at (349.0, 65.0)
- added J3: Analog, Connector_PinHeader_2.54mm:PinHeader_1x08_P2.54mm_Vertical, F.Cu at (278.0, 161.9)
- added J4: Digital, Connector_PinHeader_2.54mm:PinHeader_2x18_P2.54mm_Vertical, F.Cu at (257.6, 156.9)
- added J5: OSTOQ025450, SamacSys_Parts:SHDR2W100P0X508_1X2_1216X860X1230P, F.Cu at (296.0, 55.0)
- added J6: PWM, Connector_PinHeader_2.54mm:PinHeader_1x10_P2.54mm_Vertical, F.Cu at (332.8, 113.7)
- added J7: PWM, Connector_PinHeader_2.54mm:PinHeader_1x08_P2.54mm_Vertical, F.Cu at (305.9, 113.7)
- added J8: Communication, Connector_PinHeader_2.54mm:PinHeader_1x08_P2.54mm_Vertical, F.Cu at (283.0, 113.7)
- added J9: Conn_01x06, Connector_PinHeader_2.54mm:PinHeader_1x06_P2.54mm_Vertical, F.Cu at (278.1, 105.2)
- added JP2: Jumper_3_Open, Connector_PinHeader_2.54mm:PinHeader_1x03_P2.54mm_Vertical, F.Cu at (343.0, 179.2)
- added K1: OJE-SH-105LMH,000, SamacSys_Parts:OJESH105LMH000, F.Cu at (65.0, 82.7)
- added K10: OJE-SH-105LMH,000, SamacSys_Parts:OJESH105LMH000, F.Cu at (239.6, 82.7)
- added K11: VOR1003M4T, SamacSys_Parts:VOR1003M4T, F.Cu at (232.0, 150.0)
- added K12: VOR1003M4T, SamacSys_Parts:VOR1003M4T, F.Cu at (225.5, 150.0)
- added K13: VOR1003M4T, SamacSys_Parts:VOR1003M4T, F.Cu at (219.0, 150.0)
- added K14: VOR1003M4T, SamacSys_Parts:VOR1003M4T, F.Cu at (212.5, 150.0)
- added K15: VOR1003M4T, SamacSys_Parts:VOR1003M4T, F.Cu at (206.0, 150.0)
- added K16: VOR1003M4T, SamacSys_Parts:VOR1003M4T, F.Cu at (199.5, 150.0)
- added K17: VOR1003M4T, SamacSys_Parts:VOR1003M4T, F.Cu at (193.0, 150.0)
- added K18: VOR1003M4T, SamacSys_Parts:VOR1003M4T, F.Cu at (186.5, 150.0)
- added K19: VOR1003M4T, SamacSys_Parts:VOR1003M4T, F.Cu at (173.5, 150.0)
- added K2: OJE-SH-105LMH,000, SamacSys_Parts:OJESH105LMH000, F.Cu at (90.0, 82.7)
- added K20: VOR1003M4T, SamacSys_Parts:VOR1003M4T, F.Cu at (180.0, 150.0)
- added K3: OJE-SH-105LMH,000, SamacSys_Parts:OJESH105LMH000, F.Cu at (115.0, 82.7)
- added K4: OJE-SH-105LMH,000, SamacSys_Parts:OJESH105LMH000, F.Cu at (140.0, 82.7)
- added K5: OJE-SH-105LMH,000, SamacSys_Parts:OJESH105LMH000, F.Cu at (165.0, 82.7)
- added K6: OJE-SH-105LMH,000, SamacSys_Parts:OJESH105LMH000, F.Cu at (265.0, 82.7)
- added K7: OJE-SH-105LMH,000, SamacSys_Parts:OJESH105LMH000, F.Cu at (190.0, 82.7)
- added K8: OJE-SH-105LMH,000, SamacSys_Parts:OJESH105LMH000, F.Cu at (290.0, 82.7)
- added K9: OJE-SH-105LMH,000, SamacSys_Parts:OJESH105LMH000, F.Cu at (215.0, 82.7)
- added MH1: MountingHole_3.2mm, Arduino_MountingHole:MountingHole_3.2mm, B.Cu at (336.4, 113.7)
- added MH2: MountingHole_3.2mm, Arduino_MountingHole:MountingHole_3.2mm, B.Cu at (337.7, 161.9)
- added MH3: MountingHole_3.2mm, Arduino_MountingHole:MountingHole_3.2mm, B.Cu at (285.6, 128.9)
- added MH4: MountingHole_3.2mm, Arduino_MountingHole:MountingHole_3.2mm, B.Cu at (285.6, 156.9)
- added MH5: MountingHole_3.2mm, Arduino_MountingHole:MountingHole_3.2mm, B.Cu at (261.5, 113.7)
- added MH6: MountingHole_3.2mm, Arduino_MountingHole:MountingHole_3.2mm, B.Cu at (255.1, 161.9)
- added Q1: IRLML2060, Package_TO_SOT_SMD:SOT-23, B.Cu at (128.5, 170.8)
- added Q10: IRLML2060, Package_TO_SOT_SMD:SOT-23, F.Cu at (152.0, 78.6)
- added Q11: IRLML2060, Package_TO_SOT_SMD:SOT-23, F.Cu at (102.2, 78.7)
- added Q12: IRLML2060, Package_TO_SOT_SMD:SOT-23, F.Cu at (77.0, 78.7)
- added Q13: IRLML2060, Package_TO_SOT_SMD:SOT-23, F.Cu at (181.1, 182.0)
- added Q14: IRLML2060, Package_TO_SOT_SMD:SOT-23, F.Cu at (226.9, 78.8)
- added Q15: IRLML2060, Package_TO_SOT_SMD:SOT-23, F.Cu at (251.6, 78.7)
- added Q16: IRLML2060, Package_TO_SOT_SMD:SOT-23, F.Cu at (176.9, 78.8)
- added Q17: IRLML2060, Package_TO_SOT_SMD:SOT-23, F.Cu at (202.0, 78.7)
- added Q2: IRLML2060, Package_TO_SOT_SMD:SOT-23, B.Cu at (137.9, 170.8)
- added Q22: IRLML2060, Package_TO_SOT_SMD:SOT-23, F.Cu at (174.2, 182.0)
- added Q23: IRLML2060, Package_TO_SOT_SMD:SOT-23, F.Cu at (302.2, 78.8)
- added Q24: IRLML2060, Package_TO_SOT_SMD:SOT-23, F.Cu at (277.2, 78.6)
- added Q27: DMP6185SEQ-13, SamacSys_Parts:SOT230P700X180-4N, B.Cu at (168.0, 159.8)
- added Q28: IRLML2060, Package_TO_SOT_SMD:SOT-23, B.Cu at (167.0, 149.0)
- added Q29: IRLML2060, Package_TO_SOT_SMD:SOT-23, B.Cu at (175.2, 149.0)
- added Q3: IRLZ44N, Package_TO_SOT_THT:TO-220-3_Horizontal_TabDown, F.Cu at (74.4, 173.8)
- added Q30: DMP6185SEQ-13, SamacSys_Parts:SOT230P700X180-4N, B.Cu at (176.0, 159.8)
- added Q31: IRLML2060, Package_TO_SOT_SMD:SOT-23, B.Cu at (228.5, 146.2)
- added Q32: DMP6185SEQ-13, SamacSys_Parts:SOT230P700X180-4N, B.Cu at (229.5, 157.0)
- added Q33: IRLML2060, Package_TO_SOT_SMD:SOT-23, B.Cu at (220.5, 146.2)
- added Q34: DMP6185SEQ-13, SamacSys_Parts:SOT230P700X180-4N, B.Cu at (221.2, 157.0)
- added Q4: IRLML2060, Package_TO_SOT_SMD:SOT-23, F.Cu at (187.9, 182.0)
- added Q9: IRLML2060, Package_TO_SOT_SMD:SOT-23, F.Cu at (127.1, 78.7)
- added R1: 100R, Resistor_SMD:R_0805_2012Metric, F.Cu at (152.0, 84.1)
- added R10: 100R, Resistor_SMD:R_0805_2012Metric, F.Cu at (176.9, 84.3)
- added R102: 100R, Resistor_SMD:R_0805_2012Metric, B.Cu at (261.8, 118.8)
- added R103: 100R, Resistor_SMD:R_0805_2012Metric, B.Cu at (295.8, 118.0)
- added R104: 100R, Resistor_SMD:R_0805_2012Metric, B.Cu at (293.2, 118.0)
- added R109: 10K, Resistor_SMD:R_0805_2012Metric, B.Cu at (168.0, 152.2)
- added R11: 100K, Resistor_SMD:R_0805_2012Metric, F.Cu at (268.2, 174.0)
- added R110: 10K, Resistor_SMD:R_0805_2012Metric, B.Cu at (168.0, 154.2)
- added R111: 2K, Resistor_SMD:R_0805_2012Metric, B.Cu at (167.0, 144.0)
- added R112: 2K, Resistor_SMD:R_0805_2012Metric, B.Cu at (175.5, 144.0)
- added R113: 10K, Resistor_SMD:R_0805_2012Metric, B.Cu at (176.2, 154.2)
- added R114: 10K, Resistor_SMD:R_0805_2012Metric, B.Cu at (176.2, 152.2)
- added R115: 2K, Resistor_SMD:R_0805_2012Metric, B.Cu at (228.5, 141.2)
- added R116: 10K, Resistor_SMD:R_0805_2012Metric, B.Cu at (229.5, 149.5)
- added R117: 10K, Resistor_SMD:R_0805_2012Metric, B.Cu at (229.5, 151.5)
- added R118: 2K, Resistor_SMD:R_0805_2012Metric, B.Cu at (220.5, 141.2)
- added R119: 10K, Resistor_SMD:R_0805_2012Metric, B.Cu at (221.5, 151.5)
- added R12: 22K, Resistor_SMD:R_0805_2012Metric, F.Cu at (270.2, 174.0)
- added R120: 10K, Resistor_SMD:R_0805_2012Metric, B.Cu at (221.5, 149.5)
- added R13: 100K, Resistor_SMD:R_0805_2012Metric, F.Cu at (272.5, 174.0)
- added R14: 22K, Resistor_SMD:R_0805_2012Metric, F.Cu at (274.5, 174.0)
- added R15: 100K, Resistor_SMD:R_0805_2012Metric, F.Cu at (276.8, 174.0)
- added R16: 22K, Resistor_SMD:R_0805_2012Metric, F.Cu at (278.8, 174.0)
- added R17: 100K, Resistor_SMD:R_0805_2012Metric, F.Cu at (283.0, 174.0)
- added R18: 22K, Resistor_SMD:R_0805_2012Metric, F.Cu at (281.0, 174.0)
- added R19: 100K, Resistor_SMD:R_0805_2012Metric, F.Cu at (285.2, 174.0)
- added R2: 100R, Resistor_SMD:R_0805_2012Metric, F.Cu at (127.1, 84.2)
- added R20: 22K, Resistor_SMD:R_0805_2012Metric, F.Cu at (287.2, 174.0)
- added R21: 100K, Resistor_SMD:R_0805_2012Metric, F.Cu at (291.5, 174.0)
- added R22: 22K, Resistor_SMD:R_0805_2012Metric, F.Cu at (289.5, 174.0)
- added R23: 100K, Resistor_SMD:R_0805_2012Metric, F.Cu at (293.8, 174.0)
- added R24: 22K, Resistor_SMD:R_0805_2012Metric, F.Cu at (295.8, 174.0)
- added R25: 100K, Resistor_SMD:R_0805_2012Metric, F.Cu at (300.0, 174.0)
- added R26: 22K, Resistor_SMD:R_0805_2012Metric, F.Cu at (298.0, 174.0)
- added R27: 100K, Resistor_SMD:R_0805_2012Metric, F.Cu at (302.2, 174.0)
- added R28: 22K, Resistor_SMD:R_0805_2012Metric, F.Cu at (304.2, 174.0)
- added R29: 100K, Resistor_SMD:R_0805_2012Metric, F.Cu at (308.5, 174.0)
- added R3: 100R, Resistor_SMD:R_0805_2012Metric, F.Cu at (102.2, 84.2)
- added R30: 22K, Resistor_SMD:R_0805_2012Metric, F.Cu at (306.5, 174.0)
- added R31: R, Resistor_SMD:R_0805_2012Metric, B.Cu at (127.8, 175.0)
- added R32: R, Resistor_SMD:R_0805_2012Metric, B.Cu at (136.8, 175.0)
- added R33: 100R, Resistor_SMD:R_0805_2012Metric, F.Cu at (124.0, 175.0)
- added R34: 100R, Resistor_SMD:R_0805_2012Metric, F.Cu at (121.0, 175.0)
- added R35: 100R, Resistor_SMD:R_0805_2012Metric, F.Cu at (129.4, 175.0)
- added R36: 100R, Resistor_SMD:R_0805_2012Metric, F.Cu at (127.0, 175.0)
- added R37: R, Resistor_SMD:R_0805_2012Metric, B.Cu at (139.0, 175.0)
- added R38: 100R, Resistor_SMD:R_0805_2012Metric, F.Cu at (118.0, 174.9)
- added R39: 100R, Resistor_SMD:R_0805_2012Metric, F.Cu at (137.0, 175.0)
- added R4: 100R, Resistor_SMD:R_0805_2012Metric, F.Cu at (77.0, 84.2)
- added R40: 100R, Resistor_SMD:R_0805_2012Metric, F.Cu at (139.5, 175.0)
- added R41: 100R, Resistor_SMD:R_0805_2012Metric, F.Cu at (77.2, 173.2)
- added R42: 100K, Resistor_SMD:R_0805_2012Metric, F.Cu at (178.1, 182.0)
- added R43: 100K, Resistor_SMD:R_0805_2012Metric, F.Cu at (184.9, 182.0)
- added R44: 100K, Resistor_SMD:R_0805_2012Metric, F.Cu at (171.2, 182.0)
- added R5: 100R, Resistor_SMD:R_0805_2012Metric, F.Cu at (302.2, 84.3)
- added R56: 100R, Resistor_SMD:R_0805_2012Metric, F.Cu at (185.9, 177.3)
- added R57: 100R, Resistor_SMD:R_0805_2012Metric, F.Cu at (179.2, 177.3)
- added R6: 100R, Resistor_SMD:R_0805_2012Metric, F.Cu at (277.2, 84.1)
- added R62: 100R, Resistor_SMD:R_0805_2012Metric, F.Cu at (172.2, 177.3)
- added R65: 10K, Resistor_SMD:R_0805_2012Metric, F.Cu at (77.2, 169.3)
- added R66: 10K, Resistor_SMD:R_0805_2012Metric, F.Cu at (77.0, 82.0)
- added R67: 10K, Resistor_SMD:R_0805_2012Metric, F.Cu at (102.2, 82.0)
- added R68: 10K, Resistor_SMD:R_0805_2012Metric, F.Cu at (127.1, 82.0)
- added R69: 10K, Resistor_SMD:R_0805_2012Metric, F.Cu at (152.0, 81.9)
- added R7: 100R, Resistor_SMD:R_0805_2012Metric, F.Cu at (251.6, 84.2)
- added R70: 10K, Resistor_SMD:R_0805_2012Metric, F.Cu at (176.9, 82.0)
- added R71: 10K, Resistor_SMD:R_0805_2012Metric, F.Cu at (202.0, 82.0)
- added R72: 10K, Resistor_SMD:R_0805_2012Metric, F.Cu at (226.9, 82.0)
- added R73: 10K, Resistor_SMD:R_0805_2012Metric, F.Cu at (251.6, 82.0)
- added R74: 10K, Resistor_SMD:R_0805_2012Metric, F.Cu at (277.2, 81.9)
- added R75: 10K, Resistor_SMD:R_0805_2012Metric, F.Cu at (302.2, 82.0)
- added R76: 750R, Resistor_SMD:R_0805_2012Metric, F.Cu at (233.2, 143.0)
- added R77: 750R, Resistor_SMD:R_0805_2012Metric, F.Cu at (226.8, 143.0)
- added R78: 750R, Resistor_SMD:R_0805_2012Metric, F.Cu at (220.2, 143.0)
- added R79: 750R, Resistor_SMD:R_0805_2012Metric, F.Cu at (213.8, 143.0)
- added R8: 100R, Resistor_SMD:R_0805_2012Metric, F.Cu at (226.9, 84.3)
- added R80: 750R, Resistor_SMD:R_0805_2012Metric, F.Cu at (207.2, 143.0)
- added R81: 750R, Resistor_SMD:R_0805_2012Metric, F.Cu at (200.8, 143.0)
- added R82: 750R, Resistor_SMD:R_0805_2012Metric, F.Cu at (194.2, 143.0)
- added R83: 750R, Resistor_SMD:R_0805_2012Metric, F.Cu at (187.8, 143.0)
- added R84: 750R, Resistor_SMD:R_0805_2012Metric, F.Cu at (174.8, 143.0)
- added R85: 750R, Resistor_SMD:R_0805_2012Metric, F.Cu at (181.2, 143.0)
- added R9: 100R, Resistor_SMD:R_0805_2012Metric, F.Cu at (202.0, 84.2)
- added T7: TestPoint, SamacSys_Parts:TestPoint_Pad_0.6x0.6mm, F.Cu at (134.0, 181.2)
- added T8: TestPoint, SamacSys_Parts:TestPoint_Pad_0.6x0.6mm, F.Cu at (257.5, 175.0)
- added TTL1: TestPoint, TestPoint:TestPoint_Pad_1.0x1.0mm, F.Cu at (124.0, 170.8)
- added TTL2: TestPoint, TestPoint:TestPoint_Pad_1.0x1.0mm, F.Cu at (121.0, 170.8)
- added TTL3: TestPoint, TestPoint:TestPoint_Pad_1.0x1.0mm, F.Cu at (127.0, 170.8)
- added TTL4: TestPoint, TestPoint:TestPoint_Pad_1.0x1.0mm, F.Cu at (118.0, 170.8)
- added TTL5: TestPoint, TestPoint:TestPoint_Pad_1.0x1.0mm, F.Cu at (139.5, 170.8)
- added VC1: TestPoint, SamacSys_Parts:TestPoint_Pad_0.6x0.6mm, F.Cu at (257.5, 183.0)
- added VC2: TestPoint, SamacSys_Parts:TestPoint_Pad_0.6x0.6mm, F.Cu at (254.8, 181.8)
- added VC3: TestPoint, SamacSys_Parts:TestPoint_Pad_0.6x0.6mm, F.Cu at (257.5, 180.5)
- added VC4: TestPoint, SamacSys_Parts:TestPoint_Pad_0.6x0.6mm, F.Cu at (254.8, 179.2)
- added VC5: TestPoint, SamacSys_Parts:TestPoint_Pad_0.6x0.6mm, F.Cu at (257.5, 178.0)
- added VC6: TestPoint, SamacSys_Parts:TestPoint_Pad_0.6x0.6mm, F.Cu at (254.8, 177.0)
- added VTX1: TestPoint, TestPoint:TestPoint_Pad_1.0x1.0mm, F.Cu at (257.5, 185.8)
- added VTX2: TestPoint, TestPoint:TestPoint_Pad_1.0x1.0mm, F.Cu at (254.8, 184.2)
Routing:
- net Relay_VCC: track 0.00 -> 394.9 mm
- net VTX_2_28V: track 0.00 -> 357.5 mm, vias 0 -> 2
- net VTX_1_28V: track 0.00 -> 337.4 mm, vias 0 -> 1
- net VCAM_1 +28V: track 0.00 -> 331.0 mm, vias 0 -> 2
- net VCAM_2 +28V: track 0.00 -> 302.4 mm, vias 0 -> 2
- net Ardu_5V: track 0.00 -> 296.2 mm, vias 0 -> 2
- net VCAM_3 +28V: track 0.00 -> 281.9 mm, vias 0 -> 2
- net VDCU_28V: track 0.00 -> 274.0 mm, vias 0 -> 2
- net LD9_5V: track 0.00 -> 271.9 mm, vias 0 -> 2
- net VCAM_4 +28V: track 0.00 -> 248.6 mm, vias 0 -> 2
- net VCAM_5 +28V: track 0.00 -> 246.0 mm, vias 0 -> 2
- net /Project Architecture/Arduino Mega/*4: track 0.00 -> 238.5 mm
- net VCAM_6 +28V: track 0.00 -> 230.4 mm, vias 0 -> 2
- net Ardu_RX: track 0.00 -> 218.2 mm, vias 0 -> 1
- net EL: track 0.00 -> 216.7 mm
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- added copper zone on In2.Cu, net /Project Architecture/Connectors/EXT_5V
- added copper zone on In2.Cu, net Ardu_5V
- added copper zone on In1.Cu, net GND
- added copper zone on In2.Cu, net Relay_VCC
- added copper zone on In2.Cu, net VDCU_28V
Other:
- board outline added: 320 x 150 mm
- copper layers 6 -> 4
- board text added: "+"
- board text added: "-"
- board text added: "5V"
- board text added: "Ardu_5V"
- board text added: "EXT_5V"
- board text added: "Electronic Load"
- board text added: "JP4 is on BOT SMD"
- board text added: "LD9"
- board text added: "RX-for Ardui"
- board text added: "Relay_Vcc"
- board text added: "SW"
- board text added: "TX-by Ardui"
- board text added: "Vcc"
